Commit message: third commit

File: assets/urdf/magnet_description/capsule.urdf (robot description, URDF)
Before this commit: robot capsule, 1 links, 0 joints
Links:
- link capsule_base: geometry visual mesh filename=meshes/capsule.stl scale=0.0005 0.0005 0.0005

File: assets/urdf/magnet_description/capsule_virtual.urdf (robot description, URDF)
Before this commit: robot capsule, 1 links, 0 joints
Links:
- link capsule_base: geometry visual mesh filename=meshes/capsule.stl scale=0.0005 0.0005 0.0005

Commit message: first commit

File: assets/urdf/magnet_description/capsule.urdf (robot description, URDF)
Before this commit: robot capsule, 1 links, 0 joints
Links:
- link capsule_base: geometry collision mesh filename=meshes/capsule.stl scale=0.0005 0.0005 0.0005; visual mesh filename=meshes/capsule.stl scale=0.0005 0.0005 0.0005

File: assets/urdf/magnet_description/magnet.urdf (robot description, URDF)
Before this commit: robot magnet, 2 links, 1 joints
Links:
- link north_link: geometry visual mesh filename=meshes/north_link.STL
- link south_link: geometry visual mesh filename=meshes/south_link.STL

File: assets/urdf/magnet_description/tank1.urdf (robot description, URDF)
Before this commit: robot tank1, 1 links, 0 joints
Links:
- link tank1: mass 0.0982559999999999 -> 3.0
